File: Kicad/Rom2k40.kicad_sch (KiCad schematic)
At the start: 29 parts, among them J1 Conn_01x05_Male, J2 ~{Reset_Out}, J3 2x14 pinheader, Q1 DMG2302U, U1 74AHCT245, U2 74LVC245, U3 74LVC245, U4 74AHC1G32, U6 TLV70233_SOT23-5, U7 RP2040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

Commit message: Update README. Add EPROM pinout to sch
Other:
- title: (none) -> EPROM EMULATOR
